File: Prj 3 MCU DataLogger.kicad_pcb (KiCad board)
At the start: 0 parts

Commit message: Setup Pcbnew.
Parts:
- added BT1: Battery, Connector_PinHeader_2.54mm:PinHeader_1x02_P2.54mm_Vertical, F.Cu at (247.9, 89.3)
- added C1: 0.1uF, Capacitor_SMD:C_0805_2012Metric, F.Cu at (225.6, 99.6)
- added C2: 22pF, Capacitor_SMD:C_0805_2012Metric, F.Cu at (225.6, 96.5)
- added C3: 22pF, Capacitor_SMD:C_0805_2012Metric, F.Cu at (225.6, 93.5)
- added C4: 0.1uF, Capacitor_SMD:C_0805_2012Metric, F.Cu at (225.6, 90.5)
- added C5: 100nF, Capacitor_SMD:C_0805_2012Metric, F.Cu at (225.6, 87.5)
- added D1: LED, LED_SMD:LED_0805_2012Metric, F.Cu at (221.2, 99.5)
- added D2: LED, LED_SMD:LED_0805_2012Metric, F.Cu at (221.2, 96.5)
- added H1: MountingHole, MountingHole:MountingHole_2.1mm, F.Cu at (247.4, 111.7)
- added H2: MountingHole, MountingHole:MountingHole_2.1mm, F.Cu at (247.4, 106.0)
- added H3: MountingHole, MountingHole:MountingHole_2.1mm, F.Cu at (247.4, 100.2)
- added H4: MountingHole, MountingHole:MountingHole_2.1mm, F.Cu at (247.4, 94.5)
- added J1: Conn_01x04_Male, Connector_PinHeader_2.54mm:PinHeader_1x04_P2.54mm_Vertical, F.Cu at (210.0, 112.3)
- added J2: Conn_01x04_Male, Connector_PinHeader_2.54mm:PinHeader_1x04_P2.54mm_Vertical, F.Cu at (205.3, 112.3)
- added J3: Conn_01x09_Male, Connector_PinHeader_2.54mm:PinHeader_1x09_P2.54mm_Vertical, F.Cu at (214.6, 112.3)
- added J4: Conn_02x03_Odd_Even, Connector_PinHeader_2.54mm:PinHeader_2x03_P2.54mm_Vertical, F.Cu at (210.0, 100.0)
- added R1: 10K, Resistor_SMD:R_0805_2012Metric, F.Cu at (242.3, 113.1)
- added R2: 10K, Resistor_SMD:R_0805_2012Metric, F.Cu at (242.3, 110.2)
- added R3: 4.7K, Resistor_SMD:R_0805_2012Metric, F.Cu at (242.3, 107.2)
- added R4: 4.7K, Resistor_SMD:R_0805_2012Metric, F.Cu at (242.3, 104.3)
- added R5: 10K, Resistor_SMD:R_0805_2012Metric, F.Cu at (242.3, 101.3)
- added R6: 330, Resistor_SMD:R_0805_2012Metric, F.Cu at (242.3, 98.4)
- added R7: 330, Resistor_SMD:R_0805_2012Metric, F.Cu at (242.3, 95.4)
- added U1: 24LC1025, Package_SO:SOIC-8_5.23x5.23mm_P1.27mm, F.Cu at (234.9, 111.2)
- added U2: 24LC1025, Package_SO:SOIC-8_5.23x5.23mm_P1.27mm, F.Cu at (234.9, 104.4)
- added U3: DS1337S_, MCU DataLogger Footprints:SOIC127P600X175-8N, F.Cu at (234.9, 86.4)
- added U4: ATMEGA328P-AU, MCU DataLogger Footprints:QFP80P900X900X120-32N, F.Cu at (233.5, 95.4)
- added Y1: 16 MHz, Crystal:Crystal_SMD_5032-2Pin_5.0x3.2mm_HandSoldering, F.Cu at (224.6, 112.2)
- added Y2: 32.768 KHz, Crystal:Crystal_SMD_5032-2Pin_5.0x3.2mm_HandSoldering, F.Cu at (224.6, 107.3)
Other:
- copper layers 0 -> 2
