File: Prj 3 MCU DataLogger.kicad_pcb (KiCad board)
At the start: 4 copper layers, 55.9 x 35.5 mm, 30 parts, among them J1 Conn_01x04_Male, J2 Conn_01x04_Male, J3 Conn_01x09_Male, J4 Conn_02x03_Odd_Even, U1 24LC1025, U2 24LC1025, U3 DS1337S_, U4 ATMEGA328P-AU, Y1 16 MHz, Y2 32.768 KHz

Commit message: Created my image by using image converter with my image.
Parts:
- added G***: LOGO, Anıl's Library:anılcv_silkscreen, B.Cu at (100.5, 90.4)
- moved REF** 2.84 mm to (99.4, 78.7)
